Commit message: Switched base to Pioneer platform

File: config/kurtana.urdf (robot description, URDF)
Before this commit: robot kurtana, 45 links, 44 joints
Links:
- removed link base_footprint
- removed link ir_back
- removed link ir_left
- removed link ir_left_back
- removed link ir_left_front
- removed link ir_right
- removed link ir_right_back
- removed link ir_right_front
- removed link kurtana_rackplate_link
- removed link laser
- removed link laser_mount_link
- removed link left_front_wheel_link
- removed link left_middle_wheel_link
- removed link left_rear_wheel_link
- removed link right_front_wheel_link
- removed link right_middle_wheel_link
- removed link right_rear_wheel_link
- removed link ultrasound_front
- added link back_sonar, mass 0.0001; collision box size=0 0 0; visual mesh filename=package://p2os_urdf/meshes/p3dx_meshes/back_sonar.stl
- added link center_hubcap, mass 0.01; collision box size=0 0 0; visual mesh filename=package://p2os_urdf/meshes/p3dx_meshes/center_hubcap.stl
- added link center_wheel, mass 0.1; collision cylinder length=0.01 radius=0.0375; visual mesh filename=package://p2os_urdf/meshes/p3dx_meshes/center_wheel.stl
- added link front_sonar, mass 0.0001; collision box size=0 0 0; visual mesh filename=package://p2os_urdf/meshes/p3dx_meshes/front_sonar.stl
- added link left_hub; visual mesh filename=package://p2os_urdf/meshes/p3dx_meshes/left_hubcap.stl
- added link left_wheel_joint; visual mesh filename=package://p2os_urdf/meshes/p3dx_meshes/left_wheel.stl
- added link right_hub; visual mesh filename=package://p2os_urdf/meshes/p3dx_meshes/right_hubcap.stl
- added link right_wheel_joint; visual mesh filename=package://p2os_urdf/meshes/p3dx_meshes/right_wheel.stl
- added link swivel, mass 0.1; collision box size=0 0 0; visual mesh filename=package://p2os_urdf/meshes/p3dx_meshes/swivel.stl
- added link top_plate; visual mesh filename=package://p2os_urdf/meshes/p3dx_meshes/top.stl
- link base_link: mass 15.6 -> None; geometry visual mesh filename=package://p2os_urdf/meshes/p3dx_meshes/chassis.stl
Joints:
- removed joint base_footprint_joint
- removed joint base_ir_back
- removed joint base_ir_left
- removed joint base_ir_left_back
- removed joint base_ir_left_front
- removed joint base_ir_right
- removed joint base_ir_right_back
- removed joint base_ir_right_front
- removed joint base_ultrasound_front
- removed joint kurtana_baseplate_joint
- removed joint kurtana_laser_joint
- removed joint laser_joint
- removed joint left_front_wheel_joint
- removed joint left_middle_wheel_joint
- removed joint left_rear_wheel_joint
- removed joint right_front_wheel_joint
- removed joint right_middle_wheel_joint
- removed joint right_rear_wheel_joint
- added joint base_back_joint: type fixed, parent base_link, child back_sonar, origin xyz=0.109 0 0.209 rpy=0 0 0
- added joint base_front_joint: type fixed, parent base_link, child front_sonar, origin xyz=-0.198 0 0.208 rpy=0 0 0
- added joint base_swivel_joint: type continuous, parent base_link, child swivel, origin xyz=-0.185 0 0.055 rpy=0 0 0, limit effort=100 velocity=100
- added joint base_top_joint: type fixed, parent base_link, child top_plate, origin xyz=-0.045 0 0.234 rpy=0 0 0
- added joint center_wheel_joint: type fixed, parent center_wheel, child center_hubcap, origin xyz=-0.0035 0 -0.001 rpy=0 0 0
- added joint left_hub_joint: type fixed, parent base_link, child left_hub, origin xyz=0 0.15 0.08 rpy=0 0 0, axis 0 1 0
- added joint left_wheel_joint: type fixed, parent left_hub, child left_wheel_joint, origin xyz=0 0 0 rpy=0 0 0
- added joint right_hub_joint: type fixed, parent base_link, child right_hub, origin xyz=0 -0.15 0.08 rpy=0 0 0, axis 0 1 0
- added joint right_wheel_joint: type fixed, parent right_hub, child right_wheel_joint, origin xyz=0 0 0 rpy=0 0 0
- added joint swivel_hubcap_joint: type continuous, parent swivel, child center_wheel, origin xyz=-0.026 0 -0.016 rpy=0 0 0, axis 0 1 0, limit effort=100 velocity=100
- joint top_base_joint: child kurtana_rackplate_link -> kurtana_baseplate_link; origin xyz=0 0.0 0.0115 -> xyz=0 0.0 0.2435; parent base_link -> top_plate

Commit message: Moved back to original config

File: config/kurtana.urdf (robot description, URDF)
Before this commit: robot kurtana, 37 links, 36 joints
Links:
- link kurtana_pole_link: geometry collision box size=0.03 0.03 0.7; visual box size=0.03 0.03 0.7
Joints:
- joint kurtana_horizontal_square_bar_joint: origin xyz=0.0715 0 0.32 -> xyz=0.0715 0 0.335
- joint kurtana_microphone_joint: origin xyz=0.06 -0.055 0.37 -> xyz=0.06 -0.055 0.385
- joint kurtana_pitch_joint: origin xyz=0 0 0.008 rpy=0 0 0 -> xyz=0 0 0.008 rpy=0 0.045 0
- joint kurtana_pole_joint: origin xyz=-0.23 0 0.335 -> xyz=-0.18 0 0.35
- joint top_base_joint: origin xyz=0 0.0 0.2435 -> xyz=0 0.0 0.2115

Commit message: Finally working IKFastgit status

File: config/kurtana.urdf (robot description, URDF)
Before this commit: robot kurtana, 37 links, 36 joints
Links:
- removed link katana_base_frame
Joints:
- removed joint katana_base_frame_joint
- joint katana_gripper_tool_frame_joint: origin xyz=0 0 -0.1505 rpy=0 1.57079632679 0 -> xyz=0 0 -0.11 rpy=0 1.57079632679 0

Commit message: Assistenz robotik roboter test

File: config/kurtana.urdf (robot description, URDF)
Before this commit: robot kurtana, 36 links, 35 joints
Links:
- removed link back_sonar
- removed link center_hubcap
- removed link center_wheel
- removed link front_sonar
- removed link katana_base_link
- removed link katana_gripper_link
- removed link katana_gripper_tool_frame
- removed link katana_l_finger_link
- removed link katana_motor1_pan_link
- removed link katana_motor2_lift_link
- removed link katana_motor3_lift_link
- removed link katana_motor4_lift_link
- removed link katana_motor5_wrist_roll_link
- removed link katana_r_finger_link
- removed link left_hub
- removed link left_wheel_joint
- removed link right_hub
- removed link right_wheel_joint
- removed link swivel
- removed link top_plate
- added link base_footprint, mass 1.0; collision box size=0.001 0.001 0.001; visual box size=0.01 0.01 0.01
- added link base_laser_front_link, mass 0.001; collision cylinder length=0.09 radius=0.044; visual mesh filename=package://cob_description/meshes/sensors/sick_s300_laser.dae
- added link bl_caster_r_wheel_link, mass 0.44036; collision cylinder length=0.034 radius=0.074792; visual cylinder length=0.034 radius=0.074792
- added link bl_caster_rotation_link, mass 3.473082; collision box size=0.001 0.001 0.001; visual box size=0.001 0.001 0.001
- added link br_caster_r_wheel_link, mass 0.44036; collision cylinder length=0.034 radius=0.074792; visual cylinder length=0.034 radius=0.074792
- added link br_caster_rotation_link, mass 3.473082; collision box size=0.001 0.001 0.001; visual box size=0.001 0.001 0.001
- added link fl_caster_r_wheel_link, mass 0.44036; collision cylinder length=0.034 radius=0.074792; visual cylinder length=0.034 radius=0.074792
- added link fl_caster_rotation_link, mass 3.473082; collision box size=0.001 0.001 0.001; visual box size=0.001 0.001 0.001
- added link fr_caster_r_wheel_link, mass 0.44036; collision cylinder length=0.034 radius=0.074792; visual cylinder length=0.034 radius=0.074792
- added link fr_caster_rotation_link, mass 3.473082; collision box size=0.001 0.001 0.001; visual box size=0.001 0.001 0.001
- added link jaco_base_link; collision mesh filename=package://jaco_description/meshes/jaco_base_joint.stl; visual mesh filename=package://jaco_description/meshes/jaco_base_joint.stl
- added link jaco_finger_1_link; collision mesh filename=package://jaco_description/meshes/finger.dae; visual mesh filename=package://jaco_description/meshes/finger.dae
- added link jaco_finger_2_link; collision mesh filename=package://jaco_description/meshes/finger.dae; visual mesh filename=package://jaco_description/meshes/finger.dae
- added link jaco_finger_3_link; collision mesh filename=package://jaco_description/meshes/finger.dae; visual mesh filename=package://jaco_description/meshes/finger.dae
- added link jaco_hand_link; collision mesh filename=package://jaco_description/meshes/jaco_hand_roll_joint.stl; visual mesh filename=package://jaco_description/meshes/jaco_hand_roll_joint.stl
- added link jaco_lower_arm_link; collision mesh filename=package://jaco_description/meshes/jaco_elbow_pitch_joint.stl; visual mesh filename=package://jaco_description/meshes/jaco_elbow_pitch_joint.stl
- added link jaco_lower_arm_roll_link; collision mesh filename=package://jaco_description/meshes/jaco_elbow_roll_joint.stl; visual mesh filename=package://jaco_description/meshes/jaco_elbow_roll_joint.stl
- added link jaco_shoulder_link; collision mesh filename=package://jaco_description/meshes/jaco_shoulder_yaw_joint.s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; visual mesh filename=package://jaco_description/meshes/jaco_shoulder_yaw_joint.s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
- added link jaco_upper_arm_link; collision mesh filename=package://jaco_description/meshes/jaco_shoulder_pitch_joint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; visual mesh filename=package://jaco_description/meshes/jaco_shoulder_pitch_joint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
- added link jaco_wrist_link; collision mesh filename=package://jaco_description/meshes/jaco_wrist_roll_joint.stl; visual mesh filename=package://jaco_description/meshes/jaco_wrist_roll_joint.stl
- link base_link: mass None -> 116.0; geometry collision box size=0.62 0.48 0.17; visual box size=0.62 0.48 0.17
Joints:
- removed joint base_back_joint
- removed joint base_front_joint
- removed joint base_swivel_joint
- removed joint base_top_joint
- removed joint center_wheel_joint
- removed joint katana_gripper_joint
- removed joint katana_gripper_tool_frame_joint
- removed joint katana_l_finger_joint
- removed joint katana_motor1_pan_joint
- removed joint katana_motor2_lift_joint
- removed joint katana_motor3_lift_joint
- removed joint katana_motor4_lift_joint
- removed joint katana_motor5_wrist_roll_joint
- removed joint katana_r_finger_joint
- removed joint left_hub_joint
- removed joint left_wheel_joint
- removed joint right_hub_joint
- removed joint right_wheel_joint
- removed joint swivel_hubcap_joint
- removed joint top_base_joint
- added joint base_footprint_joint: type fixed, parent base_footprint, child base_link, origin xyz=0 0 0 rpy=0 0 0
- added joint base_laser_front_joint: type fixed, parent base_link, child base_laser_front_link, origin xyz=0.325 0.0 0.135 rpy=0 0 0, axis 0 1 0
- added joint bl_caster_r_wheel_joint: type continuous, parent bl_caster_rotation_link, child bl_caster_r_wheel_link, origin xyz=0 -0.0 0 rpy=0 0 0, axis 0 1 0, limit effort=100 velocity=100
- added joint bl_caster_rotation_joint: type continuous, parent base_link, child bl_caster_rotation_link, origin xyz=-0.235 0.185 0.075 rpy=0 0 0, axis 0 0 1, limit effort=100 velocity=100
- added joint br_caster_r_wheel_joint: type continuous, parent br_caster_rotation_link, child br_caster_r_wheel_link, origin xyz=0 -0.0 0 rpy=0 0 0, axis 0 1 0, limit effort=100 velocity=100
- added joint br_caster_rotation_joint: type continuous, parent base_link, child br_caster_rotation_link, origin xyz=-0.235 -0.185 0.075 rpy=0 0 0, axis 0 0 1, limit effort=100 velocity=100
- added joint fl_caster_r_wheel_joint: type continuous, parent fl_caster_rotation_link, child fl_caster_r_wheel_link, origin xyz=0 -0.0 0 rpy=0 0 0, axis 0 1 0, limit effort=100 velocity=100
- added joint fl_caster_rotation_joint: type continuous, parent base_link, child fl_caster_rotation_link, origin xyz=0.235 0.185 0.075 rpy=0 0 0, axis 0 0 1, limit effort=100 velocity=100
- added joint fr_caster_r_wheel_joint: type continuous, parent fr_caster_rotation_link, child fr_caster_r_wheel_link, origin xyz=0 -0.0 0 rpy=0 0 0, axis 0 1 0, limit effort=100 velocity=100
- added joint fr_caster_rotation_joint: type continuous, parent base_link, child fr_caster_rotation_link, origin xyz=0.235 -0.185 0.075 rpy=0 0 0, axis 0 0 1, limit effort=100 velocity=100
- added joint jaco_elbow_pitch_joint: type revolute, parent jaco_upper_arm_link, child jaco_lower_arm_link, origin xyz=0.41 0 0.012 rpy=0 0 0, axis 0 0 1, limit lower=-3.14159265359 upper=3.14159265359 effort=1 velocity=3.14159265359
- added joint jaco_elbow_roll_joint: type revolute, parent jaco_lower_arm_link, child jaco_lower_arm_roll_link, origin xyz=0 0.249276823007 0  rpy=-1.57079632679 0 0, axis 0 0 1, limit lower=-3.14159265359 upper=3.14159265359 effort=1 velocity=3.14159265359
- added joint jaco_finger_1_joint: type revolute, parent jaco_hand_link, child jaco_finger_1_link, origin xyz=-0.036 0.021 -0.07 rpy=0 -0.448798950513 0, axis 0 1 0, limit lower=-3.14159265359 upper=3.14159265359 effort=1 velocity=3.14159265359
- added joint jaco_finger_2_joint: type revolute, parent jaco_hand_link, child jaco_finger_2_link, origin xyz=0.036 -0 -0.07 rpy=0 -0.448798950513 -3.14159265359, axis 0 1 0, limit lower=-3.14159265359 upper=3.14159265359 effort=1 velocity=3.14159265359
- added joint jaco_finger_3_joint: type revolute, parent jaco_hand_link, child jaco_finger_3_link, origin xyz=-0.036 -0.021 -0.07 rpy=0 -0.448798950513 0, axis 0 1 0, limit lower=-3.14159265359 upper=3.14159265359 effort=1 velocity=3.14159265359
- added joint jaco_hand_roll_joint: type revolute, parent jaco_wrist_link, child jaco_hand_link, origin xyz=0 -0.186174274186 0.130360630206 rpy=0.959931088597 0 0, axis 0 0 1, limit lower=-3.14159265359 upper=3.14159265359 effort=1 velocity=3.14159265359
- added joint jaco_shoulder_pitch_joint: type revolute, parent jaco_shoulder_link, child jaco_upper_arm_link, origin xyz=0 0 0 rpy=-1.57079632679 0 0, axis 0 0 1, limit lower=-3.14159265359 upper=3.14159265359 effort=1 velocity=3.14159265359
- added joint jaco_shoulder_yaw_joint: type revolute, parent jaco_base_link, child jaco_shoulder_link, origin xyz=0 0 0.2102 rpy=0 0 0, axis 0 0 1, limit lower=-3.14159265359 upper=3.14159265359 effort=1 velocity=3.14159265359
- added joint jaco_wrist_roll_joint: type revolute, parent jaco_lower_arm_roll_link, child jaco_wrist_link, origin xyz=0 -0.0692622919853 0.0484979789618 rpy=0.959931088597 0 0, axis 0 0 1, limit lower=-3.14159265359 upper=3.14159265359 effort=1 velocity=3.14159265359
- added joint mpo_700_rack_joint: type fixed, parent base_link, child kurtana_baseplate_link, origin xyz=0 0 0.5 rpy=0 0 0
- joint kurtana_baseplate_katana_baseplate_joint: child katana_base_link -> jaco_base_link; origin xyz=0 0 0 rpy=0 0 0 -> xyz=0 0 0.05 rpy=0 0 0

Commit message: Added the distance discs to the katana wrist link

File: config/kurtana.urdf (robot description, URDF)
Before this commit: robot kurtana, 36 links, 35 joints
Links:
- added link katana_motor5_wrist_roll_discs, mass 0.05; collision cylinder length=0.025 radius=0.025; visual cylinder length=0.025 radius=0.025
- added link katana_pattern
Joints:
- added joint katana_motor5_wrist_roll_discs_joint: type fixed, parent katana_motor5_wrist_roll_link, child katana_motor5_wrist_roll_discs, origin xyz=0.0375 0 0 rpy=0 1.57079632679 0
- added joint katana_pattern_joint: type fixed, parent katana_motor4_lift_link, child katana_pattern, origin xyz=.075 -.035 0.00 rpy=1.571 -1.571 0.151

Commit message: Changed some urdf parameters for Kinect/Arm calibration

File: config/kurtana.urdf (robot description, URDF)
Before this commit: robot kurtana, 38 links, 37 joints
Links:
- link kurtana_pole_link: geometry collision box size=0.03 0.03 0.695; visual box size=0.03 0.03 0.695
Joints:
- joint kurtana_horizontal_square_bar_joint: origin xyz=0.0715 0 0.335 -> xyz=0.0715 0 0.3325
- joint kurtana_kinect_joint: origin xyz=0.03 0.0 0.018 rpy=0 0 0 -> xyz=0.0 0.0 0.0 rpy=0 0 0
- joint kurtana_microphone_joint: origin xyz=0.06 -0.055 0.385 -> xyz=0.06 -0.055 0.3825
- joint kurtana_pole_joint: origin xyz=-0.18 0 0.35 -> xyz=-0.165 0 0.3475

Commit message: first try

File: config/kurtana.urdf (robot description, URDF)
Before this commit: robot kurtana, 38 links, 37 joints
Joints:
- joint katana_l_finger_joint: limit lower=-0.44 upper=0.30 effort=0.5 velocity=0.718834 -> lower=-0.85 upper=0.30 effort=0.5 velocity=0.718834
- joint katana_r_finger_joint: limit lower=-0.44 upper=0.30 effort=0.5 velocity=0.718834 -> lower=-0.85 upper=0.30 effort=0.5 velocity=0.718834

Commit message: Shifted TCP

File: config/kurtana.urdf (robot description, URDF)
Before this commit: robot kurtana, 38 links, 37 joints
Joints:
- joint katana_gripper_tool_frame_joint: origin xyz=0 0 -0.11 rpy=0 1.57079632679 0 -> xyz=0 0 -0.19 rpy=0 1.57079632679 0
- joint katana_l_finger_joint: limit lower=-0.44 upper=0.30 effort=0.5 velocity=0.718834 -> lower=-0.85 upper=0.30 effort=0.5 velocity=1
- joint katana_r_finger_joint: limit lower=-0.44 upper=0.30 effort=0.5 velocity=0.718834 -> lower=-0.85 upper=0.30 effort=0.5 velocity=1
