Commit message: Working with gazebo jaco

File: config/kate.urdf (robot description, URDF)
Before this commit: robot kurtana, 38 links, 37 joints
Links:
- removed link back_sonar
- removed link center_hubcap
- removed link center_wheel
- removed link front_sonar
- removed link katana_base_link
- removed link katana_gripper_link
- removed link katana_gripper_tool_frame
- removed link katana_l_finger_link
- removed link katana_motor1_pan_link
- removed link katana_motor2_lift_link
- removed link katana_motor3_lift_link
- removed link katana_motor4_lift_link
- removed link katana_motor5_wrist_roll_discs
- removed link katana_motor5_wrist_roll_link
- removed link katana_pattern
- removed link katana_r_finger_link
- removed link left_hub
- removed link left_wheel_joint
- removed link right_hub
- removed link right_wheel_joint
- removed link swivel
- removed link top_plate
- added link jaco_base_link, mass 1; collision mesh filename=package://jaco_description/meshes/joint_1.dae scale=0.001 0.001 0.001; visual mesh filename=package://jaco_description/meshes/joint_1.dae scale=0.001 0.001 0.001
- added link jaco_finger_link_1, mass 0.05; collision mesh filename=package://jaco_description/meshes/finger.dae scale=1 1 1; visual mesh filename=package://jaco_description/meshes/finger.dae scale=1 1 1
- added link jaco_finger_link_2, mass 0.05; collision mesh filename=package://jaco_description/meshes/finger.dae scale=1 1 1; visual mesh filename=package://jaco_description/meshes/finger.dae scale=1 1 1
- added link jaco_finger_link_3, mass 0.05; collision mesh filename=package://jaco_description/meshes/finger.dae scale=1 1 1; visual mesh filename=package://jaco_description/meshes/finger.dae scale=1 1 1
- added link jaco_gripper_tool_frame
- added link jaco_link_1, mass 1; collision mesh filename=package://jaco_description/meshes/joint_2.dae scale=0.001 0.001 0.001; visual mesh filename=package://jaco_description/meshes/joint_2.dae scale=0.001 0.001 0.001
- added link jaco_link_2, mass 1; collision mesh filename=package://jaco_description/meshes/joint_3.dae scale=0.001 0.001 0.001; visual mesh filename=package://jaco_description/meshes/joint_3.dae scale=0.001 0.001 0.001
- added link jaco_link_3, mass 1; collision mesh filename=package://jaco_description/meshes/joint_4.dae scale=1.000 1.000 1.000; visual mesh filename=package://jaco_description/meshes/joint_4.dae scale=1.000 1.000 1.000
- added link jaco_link_4, mass 1; collision mesh filename=package://jaco_description/meshes/joint_5.dae scale=0.001 0.001 0.001; visual mesh filename=package://jaco_description/meshes/joint_5.dae scale=0.001 0.001 0.001
- added link jaco_link_5, mass 1.0; collision mesh filename=package://jaco_description/meshes/joint_6.dae scale=0.001 0.001 0.001; visual mesh filename=package://jaco_description/meshes/joint_6.dae scale=0.001 0.001 0.001
- added link jaco_link_6, mass 0.3; collision mesh filename=package://jaco_description/meshes/hand_with_noFinger.dae scale=0.001 0.001 0.001; visual mesh filename=package://jaco_description/meshes/hand_with_noFinger.dae scale=0.001 0.001 0.001
- link base_link: mass None -> 500; geometry collision mesh filename=package://p2os_urdf/meshes/p3dx_meshes/chassis.stl; visual mesh filename=package://p2os_urdf/meshes/p3dx_meshes/chassis.stl
Joints:
- removed joint base_back_joint
- removed joint base_front_joint
- removed joint base_swivel_joint
- removed joint base_top_joint
- removed joint center_wheel_joint
- removed joint katana_gripper_joint
- removed joint katana_gripper_tool_frame_joint
- removed joint katana_l_finger_joint
- removed joint katana_motor1_pan_joint
- removed joint katana_motor2_lift_joint
- removed joint katana_motor3_lift_joint
- removed joint katana_motor4_lift_joint
- removed joint katana_motor5_wrist_roll_discs_joint
- removed joint katana_motor5_wrist_roll_joint
- removed joint katana_pattern_joint
- removed joint katana_r_finger_joint
- removed joint left_hub_joint
- removed joint left_wheel_joint
- removed joint right_hub_joint
- removed joint right_wheel_joint
- removed joint swivel_hubcap_joint
- removed joint top_base_joint
- added joint base_joint: type fixed, parent base_link, child kurtana_baseplate_link, origin xyz=0 0.0 0.6115
- added joint jaco_finger_joint_1: type revolute, parent jaco_link_6, child jaco_finger_link_1, origin xyz=-0.036 -0.021 -0.09 rpy=0 0 0, axis 0 1 0, limit lower=-3.1415926535897931 upper=3.1415926535897931 effort=30 velocity=5
- added joint jaco_finger_joint_2: type revolute, parent jaco_link_6, child jaco_finger_link_2, origin xyz=-0.036 0.021 -0.09 rpy=0 0 0, axis 0 1 0, limit lower=-3.1415926535897931 upper=3.1415926535897931 effort=30 velocity=5
- added joint jaco_finger_joint_3: type revolute, parent jaco_link_6, child jaco_finger_link_3, origin xyz=0.036 -0 -0.09 rpy=0 0 3.14, axis 0 1 0, limit lower=-3.1415926535897931 upper=3.1415926535897931 effort=30 velocity=5
- added joint jaco_gripper_tool_frame_joint: type fixed, parent jaco_link_6, child jaco_gripper_tool_frame, origin xyz=0 0 0 rpy=0 -1.57079632679 1.57079632679
- added joint jaco_joint_1: type revolute, parent jaco_base_link, child jaco_link_1, origin xyz=0 0 0.2725 rpy=0 0 0, axis 0 0 -1, limit lower=-3.1415926535897931 upper=3.1415926535897931 effort=30 velocity=5
- added joint jaco_joint_2: type revolute, parent jaco_link_1, child jaco_link_2, origin xyz=0 0 0 rpy=-1.570796327 0 0, axis 0 0 1, limit lower=-3.6651914291881 upper=0.57595865315813 effort=30 velocity=5
- added joint jaco_joint_3: type revolute, parent jaco_link_2, child jaco_link_3, origin xyz=0.4100 0 0.012 rpy=0 0 0, axis 0 0 -1, limit lower=-1.221730476396 upper=4.2935099599061 effort=30 velocity=5
- added joint jaco_joint_4: type revolute, parent jaco_link_3, child jaco_link_4, origin xyz=0 0.24927682300748782 0  rpy=-1.570796327 0 0, axis 0 0 -1, limit lower=-3.1415926535897931 upper=3.1415926535897931 effort=30 velocity=5
- added joint jaco_joint_5: type revolute, parent jaco_link_4, child jaco_link_5, origin xyz=0 -0.069262292 0.048497979 rpy=0.959931089 0 0, axis 0 0 -1, limit lower=-3.1415926535897931 upper=3.1415926535897931 effort=30 velocity=5
- added joint jaco_joint_6: type revolute, parent jaco_link_5, child jaco_link_6, origin xyz=0 -0.186174274 0.13036063 rpy=-0.959931089 0 3.1415926535897931, axis 0 0 -1, limit lower=-3.5415926535897931 upper=3.5415926535897931 effort=30 velocity=5
- joint kurtana_baseplate_katana_baseplate_joint: child katana_base_link -> jaco_base_link
- joint kurtana_kinect_joint: origin xyz=0.0 0.0 0.0 rpy=0 0 0 -> xyz=0.03 0.0 0.02 rpy=0 0 0

Commit message: aalot  of changes/ cleanup

File: config/kate.urdf (robot description, URDF)
Before this commit: robot kurtana, 27 links, 26 joints
Links:
- link jaco_base_link: geometry collision mesh filename=package://jaco_description/meshes/joint_1.stl scale=0.001 0.001 0.001; visual mesh filename=package://jaco_description/meshes/joint_1.stl scale=0.001 0.001 0.001
- link jaco_finger_link_1: geometry collision mesh filename=package://jaco_description/meshes/finger.stl scale=1 1 1; visual mesh filename=package://jaco_description/meshes/finger.stl scale=1 1 1
- link jaco_finger_link_2: geometry collision mesh filename=package://jaco_description/meshes/finger.stl scale=1 1 1; visual mesh filename=package://jaco_description/meshes/finger.stl scale=1 1 1
- link jaco_finger_link_3: geometry collision mesh filename=package://jaco_description/meshes/finger.stl scale=1 1 1; visual mesh filename=package://jaco_description/meshes/finger.stl scale=1 1 1
- link jaco_link_1: geometry collision mesh filename=package://jaco_description/meshes/joint_2.stl scale=0.001 0.001 0.001; visual mesh filename=package://jaco_description/meshes/joint_2.stl scale=0.001 0.001 0.001
- link jaco_link_2: geometry collision mesh filename=package://jaco_description/meshes/joint_3.stl scale=0.001 0.001 0.001; visual mesh filename=package://jaco_description/meshes/joint_3.stl scale=0.001 0.001 0.001
- link jaco_link_3: geometry collision mesh filename=package://jaco_description/meshes/joint_4.stl scale=1.000 1.000 1.000; visual mesh filename=package://jaco_description/meshes/joint_4.stl scale=1.000 1.000 1.000
- link jaco_link_4: geometry collision mesh filename=package://jaco_description/meshes/joint_5.stl scale=0.001 0.001 0.001; visual mesh filename=package://jaco_description/meshes/joint_5.stl scale=0.001 0.001 0.001
- link jaco_link_5: geometry collision mesh filename=package://jaco_description/meshes/joint_6.stl scale=0.001 0.001 0.001; visual mesh filename=package://jaco_description/meshes/joint_6.stl scale=0.001 0.001 0.001
- link jaco_link_6: geometry collision mesh filename=package://jaco_description/meshes/hand_with_noFinger.stl scale=0.001 0.001 0.001; visual mesh filename=package://jaco_description/meshes/hand_with_noFinger.stl scale=0.001 0.001 0.001
- link kurtana_pole_link: geometry collision box size=0.03 0.03 1; visual box size=0.03 0.03 1
Joints:
- joint jaco_gripper_tool_frame_joint: origin xyz=0 0 0 rpy=0 -1.57079632679 1.57079632679 -> xyz=0 0 0 rpy=-0.2 -1.57079632679 1.57079632679
- joint kurtana_horizontal_square_bar_joint: origin xyz=0.0715 0 0.3325 -> xyz=0.0715 0 0.485
- joint kurtana_microphone_joint: origin xyz=0.06 -0.055 0.3825 -> xyz=0.06 -0.055 0.535
- joint kurtana_pole_joint: origin xyz=-0.165 0 0.3475 -> xyz=-0.25 0 0.5

Commit message: mounted arm horizontally

File: config/kate.urdf (robot description, URDF)
Before this commit: robot kurtana, 27 links, 26 joints
Joints:
- joint jaco_gripper_tool_frame_joint: origin xyz=0 0 0 rpy=-0.2 -1.57079632679 1.57079632679 -> xyz=0 0 -0.08 rpy=-0.2 -1.57079632679 1.57079632679
- joint kurtana_baseplate_katana_baseplate_joint: origin xyz=0 0 0 rpy=0 0 0 -> xyz=-0.27 0 0.27 rpy=1.57079632679 3.14159265359 1.57079632679
